Commit message: changed drone model | added PID velocity | more training

File: gym_pybullet_drones/assets/cf2x.urdf (robot description, URDF)
Before this commit: robot cf2, 6 links, 5 joints
Links:
- link base_link: geometry collision cylinder length=0.6 radius=0.5; visual mesh filename=./cf2.dae scale=8 8 8

File: gym_pybullet_drones/assets/hb.urdf (robot description, URDF)
Before this commit: robot quad, 6 links, 5 joints
Links:
- link base_link: geometry collision cylinder length=0.6 radius=0.5; visual mesh filename=./quad.obj scale=0.2 0.2 0.2
